File: Hand Mark 2 Rev 1/Hand Mark 2 Rev 1/Hand v2.0.sch (KiCad schematic (older format))
At the start: 35 parts, among them J1 Conn_ARM_JTAG_SWD_10, M1 Index_Servo, M2 Middle_Servo, M3 Ring_Servo, M4 Pinky_Servo, M5 Thumb_Servo, SW1 Power_Switch

Commit message: file rename
Parts:
- REG2: value MIC2876-5.5YMT-TR -> MIC2876-5.0YMT-T5
Changed lines of the file:
@@
 P 3800 5400
 F 0 "REG2" H 4025 5425 50  0000 C CNN
-F 1 "MIC2876-5.5YMT-TR" H 4025 5334 50  0000 C CNN
+F 1 "MIC2876-5.0YMT-T5" H 4025 5334 50  0000 C CNN
 F 2 "Package_DFN_QFN:DFN-8-1EP_2x2mm_P0.5mm_EP0.9x1.3mm" H 4000 5350 50  0001 C CNN
 F 3 "" H 4000 5350 50  0001 C CNN
